Commit message: Working robot, two wheels with a load

File: description/gazebo_control.xacro (robot description, xacro)
@@ -1,24 +1,28 @@
 <?xml version="1.0"?>
-<robot xmlns:xacro="http://www.ros.org/wiki/xacro" name="robot">
+<robot xmlns:xacro="http://www.ros.org/wiki/xacro">
     <gazebo>
-        <plugin filename="gz-sim-diff-drive-system" name="gz::sim::systems::DiffDrive">
-            <!-- WHEEL INFO -->
-            <left_joint>
-                left_wheel_joint
-            </left_joint>
-            <right_joint>
-                right_wheel_joint
-            </right_joint>
+        <plugin name="gz::sim::systems::DiffDrive" filename="gz-sim-diff-drive-system">
+            <!-- Wheel Information -->
+            <left_joint>left_wheel_joint</left_joint>
+            <right_joint>right_wheel_joint</right_joint>
             <wheel_separation>0.35</wheel_separation>
-            <wheel_diameter>0.4</wheel_diameter>
-            <!-- LIMITS -->
-            <max_wheel_torque>200</max_wheel_torque>
-            <max_wheel_acceleration>10.0</max_wheel_acceleration>
-            <!-- OUTPUT -->
-            <odometry_frame>odom</odometry_frame>
-            <robot_base_frame>base_link</robot_base_frame>
-            <publish_odom>true</publish_odom>
-            <publish_odom_tf>true</publish_odom_tf>
-            <publish_wheel_tf>true</publish_wheel_tf>
+            <wheel_radius>0.2</wheel_radius>
+            <!-- Limits -->
+            <!-- <max_wheel_torque>200</max_wheel_torque> -->
+            <max_linear_acceleration>4</max_linear_acceleration>
+            <!-- Input -->
+            <topic>/cmd_vel</topic>
+            <!-- Output -->
+            <frame_id>odom</frame_id>
+            <child_frame_id>base_link</child_frame_id>
+            <odom_topic>odom</odom_topic>
+            <odom_publisher_frequency>30</odom_publisher_frequency>
+            <tf_topic>/tf</tf_topic>
+        </plugin>
+        <plugin filename="gz-sim-joint-state-publisher-system"
+            name="gz::sim::systems::JointStatePublisher">
+            <topic>joint_states</topic>
+            <joint_name>left_wheel_joint</joint_name>
+            <joint_name>right_wheel_joint</joint_name>
         </plugin>
     </gazebo>

File: description/inertial_macros.xacro (robot description, xacro)
@@ -1,23 +1,22 @@
 <?xml version="1.0"?>
-<robot xmlns:xacro="http://www.ros.org/wiki/xacro">
-    <!-- Specify some standard inertial calculations
-    https://en.wikipedia.org/wiki/List_of_moments_of_inertia -->
+<robot xmlns:xacro="http://www.ros.org/wiki/xacro" >
+    <!-- Specify some standard inertial calculations https://en.wikipedia.org/wiki/List_of_moments_of_inertia -->
     <!-- These make use of xacro's mathematical functionality -->
     <xacro:macro name="inertial_box" params="mass x y z *origin">
         <inertial>
-            <xacro:insert_block name="origin" />
+            <xacro:insert_block name="origin"/>
             <mass value="${mass}" />
             <inertia ixx="${(1/12) * mass * (y*y+z*z)}" ixy="0.0" ixz="0.0"
-                iyy="${(1/12) * mass * (x*x+z*z)}" iyz="0.0"
-                izz="${(1/12) * mass * (x*x+y*y)}" />
+                    iyy="${(1/12) * mass * (x*x+z*z)}" iyz="0.0"
+                    izz="${(1/12) * mass * (x*x+y*y)}" />
         </inertial>
     </xacro:macro>
     <xacro:macro name="inertial_cylinder" params="mass length radius *origin">
         <inertial>
-            <xacro:insert_block name="origin" />
+            <xacro:insert_block name="origin"/>
             <mass value="${mass}" />
             <inertia ixx="${(1/12) * mass * (3*radius*radius + length*length)}" ixy="0.0" ixz="0.0"
-                iyy="${(1/12) * mass * (3*radius*radius + length*length)}" iyz="0.0"
-                izz="${(1/2) * mass * (radius*radius)}" />
+                    iyy="${(1/12) * mass * (3*radius*radius + length*length)}" iyz="0.0"
+                    izz="${(1/2) * mass * (radius*radius)}" />
         </inertial>
     </xacro:macro>

File: description/robot.urdf.xacro (robot description, xacro)
@@ -1,4 +1,11 @@
 <?xml version="1.0"?>
 <robot xmlns:xacro="http://www.ros.org/wiki/xacro" name="robot">
+    <xacro:arg name="use_ros2_control" default="false" />
     <xacro:include filename="robot_core.xacro" />
+    <xacro:if value="$(arg use_ros2_control)">
+        <xacro:include filename="ros2_control.xacro" />
+    </xacro:if>
+    <xacro:unless value="$(arg use_ros2_control)">
+        <xacro:include filename="gazebo_control.xacro" />
+    </xacro:unless>
 </robot>

File: description/robot_core.xacro (robot description, xacro)
@@ -2,4 +2,6 @@
 <robot xmlns:xacro="http://www.ros.org/wiki/xacro">
     <xacro:include filename="inertial_macros.xacro" />
+    <xacro:property name="wheel_radius" value="0.1" />
+    <xacro:property name="wheel_offset_center" value="0.2" />
     <material name="white">
         <color rgba="1 1 1 1" />
@@ -20,30 +22,64 @@
         <parent link="base_link" />
         <child link="chassis" />
-        <origin xyz="-0.15 0 0" />
+        <origin xyz="0 0 0.15" />
     </joint>
-    <!-- CHASSIS LINK -->
     <link name="chassis">
         <visual>
-            <origin xyz="0.15 0 0"></origin>
+            <origin xyz="0 0 0" />
             <geometry>
-                <box size="0.3 0.3 0.15" />
+                <box size="0.5 0.3 0.15" />
             </geometry>
             <material name="white" />
         </visual>
         <collision>
-            <origin xyz="0.15 0 0"></origin>
+            <origin xyz="0 0 0" />
             <geometry>
-                <box size="0.3 0.3 0.15" />
+                <box size="0.5 0.3 0.15" />
             </geometry>
         </collision>
-        <xacro:inertial_box mass="0.5" x="0.3" y="0.3" z="0.15">
-            <origin xyz="0.15 0 0" rpy="0 0 0" />
+        <xacro:inertial_box mass="3" x="0.5" y="0.3" z="0.15">
+            <origin xyz="0 0 0" rpy="0 0 0" />
         </xacro:inertial_box>
     </link>
+    <gazebo
+        reference="chassis">
+        <material>Gazebo/White</material>
+        <mu1>0.001</mu1>
+        <mu2>0.001</mu2>
+    </gazebo>
+    <joint name="body_joint" type="fixed">
+        <parent link="chassis" />
+        <child link="body" />
+        <origin xyz="0 0 0.15" />
+    </joint>
+    <link name="body">
+        <visual>
+            <origin xyz="0 0 0" />
+            <geometry>
+                <box size="0.3 0.15 0.15" />
+            </geometry>
+            <material name="white" />
+        </visual>
+        <collision>
+            <origin xyz="0 0 0" />
+            <geometry>
+                <box size="0.3 0.15 0.075" />
+            </geometry>
+        </collision>
+        <xacro:inertial_box mass="0.15" x="0.3" y="0.15" z="0.075">
+            <origin xyz="0 0 0" rpy="0 0 0" />
+        </xacro:inertial_box>
+    </link>
+    <gazebo
+        reference="body">
+        <material>Gazebo/Orange</material>
+        <mu1>0.001</mu1>
+        <mu2>0.001</mu2>
+    </gazebo>
     <!-- LEFT WHEEL LINK -->
     <joint name="left_wheel_joint" type="continuous">
         <parent link="base_link" />
         <child link="left_wheel" />
-        <origin xyz="0 0.175 0 " rpy="-${pi/2} 0 0" />
+        <origin xyz="-${wheel_offset_center} 0.175 0" rpy="-${pi/2} 0 0" />
         <axis xyz="0 0 1" />
     </joint>
@@ -51,24 +87,27 @@
         <visual>
             <geometry>
-                <cylinder radius="0.2" length="0.05">
-                </cylinder>
+                <cylinder radius="${wheel_radius}" length="0.05" />
             </geometry>
-            <material name="orange" />
+            <material name="blue" />
         </visual>
         <collision>
             <geometry>
-                <cylinder radius="0.2" length="0.05">
-                </cylinder>
+                <cylinder radius="${wheel_radius}" length="0.05" />
             </geometry>
         </collision>
-        <xacro:inertial_cylinder mass="1.0" length="0.05" radius="0.2">
+        <xacro:inertial_cylinder mass="0.1" length="0.05" radius="${wheel_radius}">
             <origin xyz="0 0 0" rpy="0 0 0" />
         </xacro:inertial_cylinder>
     </link>
+    <gazebo
+        reference="left_wheel">
+        <material>Gazebo/Blue</material>
+    </gazebo>
     <!-- RIGHT WHEEL LINK -->
-    <joint name="right_wheel_joint" type="continuous">
+    <joint name="right_wheel_joint"
+        type="continuous">
         <parent link="base_link" />
         <child link="right_wheel" />
-        <origin xyz="0 -0.175 0 " rpy="${pi/2} 0 0" />
+        <origin xyz="-${wheel_offset_center} -0.175 0" rpy="${pi/2} 0 0" />
         <axis xyz="0 0 -1" />
     </joint>
@@ -76,18 +115,79 @@
         <visual>
             <geometry>
-                <cylinder radius="0.2" length="0.05">
-                </cylinder>
+                <cylinder radius="${wheel_radius}" length="0.05" />
             </geometry>
-            <material name="orange" />
+            <material name="blue" />
         </visual>
         <collision>
             <geometry>
-                <cylinder radius="0.2" length="0.05">
-                </cylinder>
+                <cylinder radius="${wheel_radius}" length="0.05" />
             </geometry>
         </collision>
-        <xacro:inertial_cylinder mass="1.0" length="0.05" radius="0.2">
+        <xacro:inertial_cylinder mass="0.1" length="0.05" radius="${wheel_radius}">
             <origin xyz="0 0 0" rpy="0 0 0" />
         </xacro:inertial_cylinder>
     </link>
+    <gazebo
+        reference="right_wheel">
+        <material>Gazebo/Blue</material>
+    </gazebo>
+    <!-- FRONT LEFT WHEEL LINK-->
+    <joint name="front_left_wheel_joint" type="continuous">
+        <parent link="base_link" />
+        <child link="front_left_wheel" />
+        <origin xyz="${wheel_offset_center} 0.175 0" rpy="-${pi/2} 0 0" />
+        <axis xyz="0 0 1" />
+    </joint>
+    <link name="front_left_wheel">
+        <visual>
+            <geometry>
+                <cylinder radius="${wheel_radius}" length="0.05" />
+            </geometry>
+            <material name="blue" />
+        </visual>
+        <collision>
+            <geometry>
+                <cylinder radius="${wheel_radius}" length="0.05" />
+            </geometry>
+        </collision>
+        <xacro:inertial_cylinder mass="0.1" length="0.05" radius="${wheel_radius}">
+            <origin xyz="0 0 0" rpy="0 0 0" />
+        </xacro:inertial_cylinder>
+    </link>
+    <gazebo
+        reference="front_left_wheel">
+        <material>Gazebo/Blue</material>
+        <mu1>0.001</mu1>
+        <mu2>0.001</mu2>
+    </gazebo>
+    <!-- FRONT RIGHT WHEEL LINK-->
+    <joint name="front_right_wheel_joint"
+        type="continuous">
+        <parent link="base_link" />
+        <child link="front_right_wheel" />
+        <origin xyz="${wheel_offset_center} -0.175 0" rpy="${pi/2} 0 0" />
+        <axis xyz="0 0 -1" />
+    </joint>
+    <link name="front_right_wheel">
+        <visual>
+            <geometry>
+                <cylinder radius="${wheel_radius}" length="0.05" />
+            </geometry>
+            <material name="blue" />
+        </visual>
+        <collision>
+            <geometry>
+                <cylinder radius="${wheel_radius}" length="0.05" />
+            </geometry>
+        </collision>
+        <xacro:inertial_cylinder mass="0.1" length="0.05" radius="${wheel_radius}">
+            <origin xyz="0 0 0" rpy="0 0 0" />
+        </xacro:inertial_cylinder>
+    </link>
+    <gazebo
+        reference="front_right_wheel">
+        <material>Gazebo/Blue</material>
+        <mu1>0.001</mu1>
+        <mu2>0.001</mu2>
+    </gazebo>
 </robot>
