Commit message: Added a Lidar with new Gazebo considerations in mind, updated README

File: description/robot.urdf.xacro (robot description, xacro)
@@ -9,3 +9,4 @@
         <xacro:include filename="gazebo_control.xacro" />
     </xacro:unless>
+    <xacro:include filename="lidar.xacro" />
 </robot>

File: description/robot_core.xacro (robot description, xacro)
@@ -45,33 +45,4 @@
         reference="chassis">
         <material>Gazebo/White</material>
-        <mu1>0.001</mu1>
-        <mu2>0.001</mu2>
-    </gazebo>
-    <joint name="body_joint" type="fixed">
-        <parent link="chassis" />
-        <child link="body" />
-        <origin xyz="0 0 0.15" />
-    </joint>
-    <link name="body">
-        <visual>
-            <origin xyz="0 0 0" />
-            <geometry>
-                <box size="0.3 0.15 0.15" />
-            </geometry>
-            <material name="white" />
-        </visual>
-        <collision>
-            <origin xyz="0 0 0" />
-            <geometry>
-                <box size="0.3 0.15 0.075" />
-            </geometry>
-        </collision>
-        <xacro:inertial_box mass="0.15" x="0.3" y="0.15" z="0.075">
-            <origin xyz="0 0 0" rpy="0 0 0" />
-        </xacro:inertial_box>
-    </link>
-    <gazebo
-        reference="body">
-        <material>Gazebo/Orange</material>
         <mu1>0.001</mu1>
         <mu2>0.001</mu2>
@@ -133,5 +104,5 @@
     </gazebo>
     <!-- FRONT LEFT WHEEL LINK-->
-    <joint name="front_left_wheel_joint" type="continuous">
+    <joint name="front_left_wheel_joint" type="fixed">
         <parent link="base_link" />
         <child link="front_left_wheel" />
@@ -163,5 +134,5 @@
     <!-- FRONT RIGHT WHEEL LINK-->
     <joint name="front_right_wheel_joint"
-        type="continuous">
+        type="fixed">
         <parent link="base_link" />
         <child link="front_right_wheel" />
